Commit message: Propellers are actually continuous joints

File: urdf/custom_iris.xacro (robot description, xacro)
@@ -58,7 +58,6 @@
         </collision>
     </link>
-    <joint name="rotor_0_joint" type="revolute">
-        <axis xyz="0 0 1"/>
-        <limit lower="-1000000000000" upper="100000000000" effort="10" velocity="30"/>
+    <joint name="rotor_0_joint" type="continuous">
+        <axis xyz="0 0 1"/>
         <origin xyz="0.13 -0.22 0.023" rpy="0 0 0" />
         <parent link="base_link"/>
@@ -85,7 +84,6 @@
         </collision>
     </link>
-    <joint name="rotor_1_joint" type="revolute">
-        <axis xyz="0 0 1"/>
-        <limit lower="-1000000000000" upper="100000000000" effort="10" velocity="30"/>
+    <joint name="rotor_1_joint" type="continuous">
+        <axis xyz="0 0 1"/>
         <origin xyz="-0.13 0.22 0.023" rpy="0 0 0" />
         <parent link="base_link"/>
@@ -112,7 +110,6 @@
         </collision>
     </link>
-    <joint name="rotor_2_joint" type="revolute">
-        <axis xyz="0 0 1"/>
-        <limit lower="-1000000000000" upper="100000000000" effort="10" velocity="30"/>
+    <joint name="rotor_2_joint" type="continuous">
+        <axis xyz="0 0 1"/>
         <origin xyz="0.13 0.22 0.023" rpy="0 0 0" />
         <parent link="base_link"/>
@@ -139,7 +136,6 @@
         </collision>
     </link>
-    <joint name="rotor_3_joint" type="revolute">
-        <axis xyz="0 0 1"/>
-        <limit lower="-1000000000000" upper="100000000000" effort="10" velocity="30"/>
+    <joint name="rotor_3_joint" type="continuous">
+        <axis xyz="0 0 1"/>
         <origin xyz="-0.13 -0.22 0.023" rpy="0 0 0" />
         <parent link="base_link"/>

Commit message: PX4-custom urdf now communicating successfully. That required an amazing amount of debugging... Phew! :beers:

File: urdf/custom_iris.xacro (robot description, xacro)
@@ -28,5 +28,5 @@
             <origin xyz="0 0 0" rpy="0 0 0"/>
             <geometry>
-                <mesh filename="package://uav_inspections_ros2/meshes/iris.stl"/>
+                <box size="0.47 0.47 0.11"/>
             </geometry>
         </collision>
@@ -54,5 +54,6 @@
             <origin xyz="0 0 0" rpy="0 0 0"/>
             <geometry>
-                <mesh filename="package://uav_inspections_ros2/meshes/iris_prop_ccw.stl"/>
+                <cylinder length="0.005" radius="0.128" />
+                <!-- <mesh filename="package://uav_inspections_ros2/meshes/iris_prop_ccw.stl"/> -->
             </geometry>
         </collision>
@@ -80,5 +81,6 @@
             <origin xyz="0 0 0" rpy="0 0 0"/>
             <geometry>
-                <mesh filename="package://uav_inspections_ros2/meshes/iris_prop_ccw.stl"/>
+                <cylinder length="0.005" radius="0.128" />
+                <!-- <mesh filename="package://uav_inspections_ros2/meshes/iris_prop_ccw.stl"/> -->
             </geometry>
         </collision>
@@ -106,5 +108,6 @@
             <origin xyz="0 0 0" rpy="0 0 0"/>
             <geometry>
-                <mesh filename="package://uav_inspections_ros2/meshes/iris_prop_cw.stl"/>
+                <cylinder length="0.005" radius="0.128" />
+                <!-- <mesh filename="package://uav_inspections_ros2/meshes/iris_prop_cw.stl"/> -->
             </geometry>
         </collision>
@@ -132,5 +135,6 @@
             <origin xyz="0 0 0" rpy="0 0 0"/>
             <geometry>
-                <mesh filename="package://uav_inspections_ros2/meshes/iris_prop_cw.stl"/>
+                <cylinder length="0.005" radius="0.128" />
+                <!-- <mesh filename="package://uav_inspections_ros2/meshes/iris_prop_cw.stl"/> -->
             </geometry>
         </collision>
@@ -149,15 +153,53 @@
       <child link="camera_link" />
     </joint>
-    <link name="imu_link"/>
-    <joint name="imu_joint" type="fixed">
-      <origin xyz="0 0 0" rpy="0 0 0" />
+    <link name="imu_link">
+        <inertial>
+            <mass value="0.015" />
+            <origin xyz="0 0 0"/>
+            <inertia ixx="1e-05" ixy="0.0" ixz="0.0" iyy="1e-05" iyz="0.0" izz="1e-05" />
+        </inertial>
+        <visual>
+            <origin xyz="0 0 0" rpy="0 0 0"/>
+            <geometry>
+                <cylinder length="0.01" radius="0.002" />
+            </geometry>
+        </visual>
+        <collision>
+            <origin xyz="0 0 0" rpy="0 0 0"/>
+            <geometry>
+                <cylinder length="0.01" radius="0.002" />
+            </geometry>
+        </collision>
+    </link>
+    <joint name="imu_joint" type="revolute">
+      <origin xyz="0.1 0 0" rpy="0 0 0" />
       <parent link="base_link"/>
       <child link="imu_link" />
-    </joint>
-    <link name="gps_link"/>
-    <joint name="gps_joint" type="fixed">
-      <origin xyz="0 0 0" rpy="0 0 0" />
+      <limit effort="0" velocity="0" lower="0" upper="0" />
+    </joint>
+    <link name="gps_link">
+        <inertial>
+            <mass value="0.015" />
+            <origin xyz="0 0 0"/>
+            <inertia ixx="1e-05" ixy="0.0" ixz="0.0" iyy="1e-05" iyz="0.0" izz="1e-05" />
+        </inertial>
+        <visual>
+            <origin xyz="0 0 0" rpy="0 0 0"/>
+            <geometry>
+                <cylinder length="0.01" radius="0.002" />
+            </geometry>
+        </visual>
+        <collision>
+            <origin xyz="0 0 0" rpy="0 0 0"/>
+            <geometry>
+                <cylinder length="0.01" radius="0.002" />
+            </geometry>
+        </collision>
+    </link>
+    <joint name="gps_joint" type="revolute">
+      <origin xyz="-0.1 0 0" rpy="0 0 0" />
       <parent link="base_link"/>
       <child link="gps_link" />
+      <limit effort="0" velocity="0" lower="0" upper="0" />
     </joint>
     <link name="magnetometer_link"/>
@@ -173,5 +215,5 @@
       <child link="barometer_link" />
     </joint>
-    <!-- Gazebo -->
+    <!-- General Gazebo -->
     <gazebo reference="chassis_link">
        <material>Gazebo/Grey</material>
@@ -189,4 +231,5 @@
        <material>Gazebo/Yellow</material>
     </gazebo>
+    <!-- ROS2 Gazebo -->
     <gazebo>
     <plugin name="ground_truth_odom" filename="libgazebo_ros_p3d.so">
@@ -195,5 +238,5 @@
         </ros>
         <body_name>base_link</body_name>
-        <frame_name>chassis_link</frame_name>
+        <frame_name>world</frame_name>
         <update_rate>1</update_rate>
         <xyz_offset>0 0 0</xyz_offset>
@@ -206,5 +249,5 @@
         <always_on>true</always_on>
         <update_rate>30</update_rate>
-      <camera name="camera">
+        <camera name="camera">
         <horizontal_fov>1.2</horizontal_fov>
         <image>
@@ -235,18 +278,19 @@
     </sensor>
     </gazebo>
-    <gazebo reference="imu_link">
-    <plugin name='rotors_gazebo_imu_plugin' filename='libgazebo_imu_plugin.so'>
-      <robotNamespace/>
-      <linkName>/imu_link</linkName>
-      <imuTopic>/imu</imuTopic>
-      <gyroscopeNoiseDensity>0.00018665</gyroscopeNoiseDensity>
-      <gyroscopeRandomWalk>3.8785e-05</gyroscopeRandomWalk>
-      <gyroscopeBiasCorrelationTime>1000.0</gyroscopeBiasCorrelationTime>
-      <gyroscopeTurnOnBiasSigma>0.0087</gyroscopeTurnOnBiasSigma>
-      <accelerometerNoiseDensity>0.00186</accelerometerNoiseDensity>
-      <accelerometerRandomWalk>0.006</accelerometerRandomWalk>
-      <accelerometerBiasCorrelationTime>300.0</accelerometerBiasCorrelationTime>
-      <accelerometerTurnOnBiasSigma>0.196</accelerometerTurnOnBiasSigma>
-    </plugin>
+    <gazebo>
+    <plugin name="gazebo_ros_joint_state_publisher" filename="libgazebo_ros_joint_state_publisher.so">
+        <ros>
+          <namespace></namespace>
+        </ros>
+        <update_rate>2</update_rate>
+        <joint_name>rotor_0_joint</joint_name>
+        <joint_name>rotor_1_joint</joint_name>
+        <joint_name>rotor_2_joint</joint_name>
+        <joint_name>rotor_3_joint</joint_name>
+        <joint_name>imu_joint</joint_name>
+        <joint_name>gps_joint</joint_name>
+    </plugin>
+    </gazebo>
+    <!-- <gazebo reference="imu_link"> -->
     <!-- <sensor name="imu" type="imu"> -->
     <!-- <always_on>true</always_on> -->
@@ -260,65 +304,6 @@
     <!-- </plugin> -->
     <!-- </sensor> -->
-    </gazebo>
-    <gazebo reference="gps_link">
-    <sensor name="gps" type="gps">
-        <pose>0 0 0 0 0 0</pose>
-        <update_rate>5.0</update_rate>
-        <always_on>true</always_on>
-        <visualize>false</visualize>
-        <!-- GpsSensor noise currently not used -->
-        <!-- <gps>
-          <position_sensing>
-            <horizontal>
-              <noise type="gaussian_quantized">
-                <mean>0</mean>
-                <stddev>1</stddev>
-                <bias_mean>3</bias_mean>
-                <bias_stddev>1</bias_stddev>
-                <precision>0.5</precision>
-              </noise>
-            </horizontal>
-            <vertical>
-              <noise type="gaussian_quantized">
-                <mean>0</mean>
-                <stddev>1</stddev>
-                <bias_mean>3</bias_mean>
-                <bias_stddev>1</bias_stddev>
-                <precision>1.0</precision>
-              </noise>
-            </vertical>
-          </position_sensing>
-          <velocity_sensing>
-            <horizontal>
-              <noise type="gaussian_quantized">
-                <mean>0</mean>
-                <stddev>0.1</stddev>
-                <bias_mean>0.1</bias_mean>
-                <bias_stddev>0.1</bias_stddev>
-                <precision>0.1</precision>
-              </noise>
-            </horizontal>
-            <vertical>
-              <noise type="gaussian_quantized">
-                <mean>0</mean>
-                <stddev>0.2</stddev>
-                <bias_mean>0.2</bias_mean>
-                <bias_stddev>0.2</bias_stddev>
-                <precision>0.2</precision>
-              </noise>
-            </vertical>
-          </velocity_sensing>
-        </gps> -->
-        <plugin name="gps_plugin" filename="libgazebo_gps_plugin.so">
-          <robotNamespace></robotNamespace>
-          <gpsNoise>true</gpsNoise>
-          <gpsXYRandomWalk>2.0</gpsXYRandomWalk>
-          <gpsZRandomWalk>4.0</gpsZRandomWalk>
-          <gpsXYNoiseDensity>2.0e-4</gpsXYNoiseDensity>
-          <gpsZNoiseDensity>4.0e-4</gpsZNoiseDensity>
-          <gpsVXYNoiseDensity>0.2</gpsVXYNoiseDensity>
-          <gpsVZNoiseDensity>0.4</gpsVZNoiseDensity>
-        </plugin>
-      </sensor>
+    <!-- </gazebo> -->
+    <!-- <gazebo reference="gps_link"> -->
     <!-- <sensor name="gps" type="gps"> -->
           <!-- <always_on>true</always_on> -->
@@ -347,6 +332,86 @@
           <!-- </plugin> -->
         <!-- </sensor> -->
-    </gazebo>
-    <gazebo reference="rotor_0">
+    <!-- </gazebo> -->
+    <!-- PX4 Gazebo -->
+    <gazebo reference="gps_link">
+        <sensor name="gps" type="gps">
+        <update_rate>5</update_rate>
+        <always_on>true</always_on>
+        <visualize>false</visualize>
+        <!-- GpsSensor noise currently not used -->
+        <!-- <gps> -->
+          <!-- <position_sensing> -->
+            <!-- <horizontal> -->
+              <!-- <noise type="gaussian_quantized"> -->
+                <!-- <mean>0</mean> -->
+                <!-- <stddev>1</stddev> -->
+                <!-- <bias_mean>3</bias_mean> -->
+                <!-- <bias_stddev>1</bias_stddev> -->
+                <!-- <precision>0.5</precision> -->
+              <!-- </noise> -->
+            <!-- </horizontal> -->
+            <!-- <vertical> -->
+              <!-- <noise type="gaussian_quantized"> -->
+                <!-- <mean>0</mean> -->
+                <!-- <stddev>1</stddev> -->
+                <!-- <bias_mean>3</bias_mean> -->
+                <!-- <bias_stddev>1</bias_stddev> -->
+                <!-- <precision>1.0</precision> -->
+              <!-- </noise> -->
+            <!-- </vertical> -->
+          <!-- </position_sensing> -->
+          <!-- <velocity_sensing> -->
+            <!-- <horizontal> -->
+              <!-- <noise type="gaussian_quantized"> -->
+                <!-- <mean>0</mean> -->
+                <!-- <stddev>0.1</stddev> -->
+                <!-- <bias_mean>0.1</bias_mean> -->
+                <!-- <bias_stddev>0.1</bias_stddev> -->
+                <!-- <precision>0.1</precision> -->
+              <!-- </noise> -->
+            <!-- </horizontal> -->
+            <!-- <vertical> -->
+              <!-- <noise type="gaussian_quantized"> -->
+                <!-- <mean>0</mean> -->
+                <!-- <stddev>0.2</stddev> -->
+                <!-- <bias_mean>0.2</bias_mean> -->
+                <!-- <bias_stddev>0.2</bias_stddev> -->
+                <!-- <precision>0.2</precision> -->
+              <!-- </noise> -->
+            <!-- </vertical> -->
+          <!-- </velocity_sensing> -->
+        <!-- </gps>  -->
+        <plugin name="gps_plugin" filename="libgazebo_gps_plugin.so">
+          <robotNamespace></robotNamespace>
+          <topic>/gps</topic>
+          <linkName>gps_link</linkName>
+          <update_rate>5</update_rate>
+          <always_on>true</always_on>
+          <gpsNoise>true</gpsNoise>
+          <gpsXYRandomWalk>2.0</gpsXYRandomWalk>
+          <gpsZRandomWalk>4.0</gpsZRandomWalk>
+          <gpsXYNoiseDensity>2.0e-4</gpsXYNoiseDensity>
+          <gpsZNoiseDensity>4.0e-4</gpsZNoiseDensity>
+          <gpsVXYNoiseDensity>0.2</gpsVXYNoiseDensity>
+          <gpsVZNoiseDensity>0.4</gpsVZNoiseDensity>
+        </plugin>
+      </sensor>
+    </gazebo>
+    <gazebo>
+    <plugin name='rotors_gazebo_imu_plugin' filename='libgazebo_imu_plugin.so'>
+        <robotNamespace></robotNamespace>
+      <linkName>imu_link</linkName>
+      <imuTopic>/imu</imuTopic>
+      <gyroscopeNoiseDensity>0.00018665</gyroscopeNoiseDensity>
+      <gyroscopeRandomWalk>3.8785e-05</gyroscopeRandomWalk>
+      <gyroscopeBiasCorrelationTime>1000.0</gyroscopeBiasCorrelationTime>
+      <gyroscopeTurnOnBiasSigma>0.0087</gyroscopeTurnOnBiasSigma>
+      <accelerometerNoiseDensity>0.00186</accelerometerNoiseDensity>
+      <accelerometerRandomWalk>0.006</accelerometerRandomWalk>
+      <accelerometerBiasCorrelationTime>300.0</accelerometerBiasCorrelationTime>
+      <accelerometerTurnOnBiasSigma>0.196</accelerometerTurnOnBiasSigma>
+    </plugin>
+    </gazebo>
+    <gazebo>
     <plugin name='front_right_motor_model' filename='libgazebo_motor_model.so'>
       <robotNamespace/>
@@ -367,5 +432,5 @@
     </plugin>
     </gazebo>
-    <gazebo reference="rotor_1">
+    <gazebo>
     <plugin name='back_left_motor_model' filename='libgazebo_motor_model.so'>
       <robotNamespace/>
@@ -386,5 +451,5 @@
     </plugin>
     </gazebo>
-    <gazebo reference="rotor_2">
+    <gazebo>
     <plugin name='front_left_motor_model' filename='libgazebo_motor_model.so'>
       <robotNamespace/>
@@ -405,5 +470,5 @@
     </plugin>
     </gazebo>
-    <gazebo reference="rotor_3">
+    <gazebo>
     <plugin name='back_right_motor_model' filename='libgazebo_motor_model.so'>
       <robotNamespace/>
@@ -424,5 +489,5 @@
     </plugin>
     </gazebo>
-    <gazebo reference="barometer_link">
+    <gazebo>
     <plugin name='barometer_plugin' filename='libgazebo_barometer_plugin.so'>
       <robotNamespace/>
@@ -432,5 +497,5 @@
     </plugin>
     </gazebo>
-    <gazebo reference="magnetometer_link">
+    <gazebo>
     <plugin name='magnetometer_plugin' filename='libgazebo_magnetometer_plugin.so'>
       <robotNamespace/>
@@ -442,46 +507,8 @@
     </plugin>
     </gazebo>
-    <!-- Transmissions (not sure if needed yet)-->
-  <!-- <transmission name="rotor_0_trans"> -->
-    <!-- <type>transmission_interface/SimpleTransmission</type> -->
-    <!-- <actuator name="rotor_0"> -->
-      <!-- <mechanicalReduction>1</mechanicalReduction> -->
-    <!-- </actuator> -->
-    <!-- <joint name="rotor_0_joint"> -->
-      <!-- <hardwareInterface>EffortJointInterface</hardwareInterface> -->
-    <!-- </joint> -->
-  <!-- </transmission> -->
-  <!-- <transmission name="rotor_1_trans"> -->
-    <!-- <type>transmission_interface/SimpleTransmission</type> -->
-    <!-- <actuator name="rotor_1"> -->
-      <!-- <mechanicalReduction>1</mechanicalReduction> -->
-    <!-- </actuator> -->
-    <!-- <joint name="rotor_1_joint"> -->
-      <!-- <hardwareInterface>EffortJointInterface</hardwareInterface> -->
-    <!-- </joint> -->
-  <!-- </transmission> -->
-  <!-- <transmission name="rotor_2_trans"> -->
-    <!-- <type>transmission_interface/SimpleTransmission</type> -->
-    <!-- <actuator name="rotor_2"> -->
-      <!-- <mechanicalReduction>1</mechanicalReduction> -->
-    <!-- </actuator> -->
-    <!-- <joint name="rotor_2_joint"> -->
-      <!-- <hardwareInterface>EffortJointInterface</hardwareInterface> -->
-    <!-- </joint> -->
-  <!-- </transmission> -->
-  <!-- <transmission name="rotor_3_trans"> -->
-    <!-- <type>transmission_interface/SimpleTransmission</type> -->
-    <!-- <actuator name="rotor_3"> -->
-      <!-- <mechanicalReduction>1</mechanicalReduction> -->
-    <!-- </actuator> -->
-    <!-- <joint name="rotor_3_joint"> -->
-      <!-- <hardwareInterface>EffortJointInterface</hardwareInterface> -->
-    <!-- </joint> -->
-  <!-- </transmission> -->
     <gazebo>
     <plugin name='mavlink_interface' filename='libgazebo_mavlink_interface.so'>
       <robotNamespace/>
       <imuSubTopic>/imu</imuSubTopic>
-      <gpsSubTopic>/gps</gpsSubTopic>
       <magSubTopic>/mag</magSubTopic>
       <baroSubTopic>/baro</baroSubTopic>
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
Commit message: Added complete depth camera integration

File: urdf/custom_iris.xacro (robot description, xacro)
@@ -149,7 +149,13 @@
     <link name="camera_link"/>
     <joint name="camera_joint" type="fixed">
-      <origin xyz="0.05 0 -0.05" rpy="0 0 0" />
+      <origin xyz="0.15 0 -0.01" rpy="0 0 0" />
       <parent link="base_link"/>
       <child link="camera_link" />
+    </joint>
+    <link name="camera_optical_link"/>
+    <joint name="camera_optical_joint" type="fixed">
+      <origin xyz="0 0 0" rpy="-1.57079632679 0 -1.57079632679"/>
+      <parent link="camera_link"/>
+      <child link="camera_optical_link" />
     </joint>
     <link name="imu_link">
@@ -272,5 +278,5 @@
       <plugin name="simulated_camera" filename="libgazebo_ros_camera.so">
         <camera_name>camera</camera_name>
-        <frame_name>camera_link</frame_name>
+        <frame_name>camera_optical_link</frame_name>
         <hack_baseline>0.07</hack_baseline>
         <min_depth>0.001</min_depth>

Commit message: Added a commented out ros2 control plugin which is currently not working

File: urdf/custom_iris.xacro (robot description, xacro)
@@ -298,4 +298,25 @@
     </plugin>
     </gazebo>
+    <!-- <ros2_control name="GazeboSystem" type="system"> -->
+        <!-- <hardware> -->
+            <!-- <plugin>gazebo_ros2_control/GazeboSystem</plugin> -->
+        <!-- </hardware> -->
+        <!-- <joint name="virtual_joint"> -->
+            <!-- <command_interface name="position"> -->
+                <!-- <param name="min">-9999</param> -->
+                <!-- <param name="max">9999</param> -->
+            <!-- </command_interface> -->
+            <!-- <state_interface name="position"/> -->
+            <!-- <state_interface name="velocity"/> -->
+            <!-- <state_interface name="effort"/> -->
+        <!-- </joint> -->
+    <!-- </ros2_control> -->
+    <!-- <gazebo> -->
+    <!-- <plugin name="gazebo_ros2_control" filename="libgazebo_ros2_control.so"> -->
+      <!-- <robot_param>robot_description</robot_param> -->
+      <!-- <robot_param_node>robot_state_publisher</robot_param_node> -->
+      <!-- <parameters>$(find uav_inspections_ros2)/config/uav_ros_controllers.yaml</parameters> -->
+    <!-- </plugin> -->
+    <!-- </gazebo> -->
     <!-- <gazebo reference="imu_link"> -->
     <!-- <sensor name="imu" type="imu"> -->

Commit message: Changed to a fake controller for now

File: urdf/custom_iris.xacro (robot description, xacro)
@@ -254,5 +254,5 @@
     <sensor type="depth" name="camera">
         <always_on>true</always_on>
-        <update_rate>30</update_rate>
+        <update_rate>15</update_rate>
         <camera name="camera">
         <horizontal_fov>1.2</horizontal_fov>
@@ -266,5 +266,5 @@
         <clip>
           <near>0.02</near>
-          <far>100</far>
+          <far>12</far>
         </clip>
         <distortion>
@@ -298,18 +298,16 @@
     </plugin>
     </gazebo>
-    <!-- <ros2_control name="GazeboSystem" type="system"> -->
-        <!-- <hardware> -->
+    <ros2_control name="GazeboSystem" type="system">
+        <hardware>
             <!-- <plugin>gazebo_ros2_control/GazeboSystem</plugin> -->
-        <!-- </hardware> -->
-        <!-- <joint name="virtual_joint"> -->
-            <!-- <command_interface name="position"> -->
-                <!-- <param name="min">-9999</param> -->
-                <!-- <param name="max">9999</param> -->
-            <!-- </command_interface> -->
-            <!-- <state_interface name="position"/> -->
-            <!-- <state_interface name="velocity"/> -->
-            <!-- <state_interface name="effort"/> -->
-        <!-- </joint> -->
-    <!-- </ros2_control> -->
+            <plugin>fake_components/GenericSystem</plugin>
+        </hardware>
+        <joint name="virtual_joint">
+            <command_interface name="position"/>
+            <state_interface name="position"/>
+            <state_interface name="velocity"/>
+            <state_interface name="effort"/>
+        </joint>
+    </ros2_control>
     <!-- <gazebo> -->
     <!-- <plugin name="gazebo_ros2_control" filename="libgazebo_ros2_control.so"> -->
