Commit message: Minor urdf changes, mainly for higher sensor rates

File: urdf/custom_iris.xacro (robot description, xacro)
@@ -245,5 +245,5 @@
         <body_name>base_link</body_name>
         <frame_name>odom</frame_name>
-        <update_rate>30</update_rate>
+        <update_rate>10</update_rate>
         <xyz_offset>0 0 0</xyz_offset>
         <rpy_offset>0 0 0</rpy_offset>
@@ -254,5 +254,5 @@
     <sensor type="depth" name="camera">
         <always_on>true</always_on>
-        <update_rate>15</update_rate>
+        <update_rate>10</update_rate>
         <camera name="camera">
         <horizontal_fov>1.2</horizontal_fov>
@@ -303,10 +303,10 @@
             <plugin>fake_components/GenericSystem</plugin>
         </hardware>
-        <joint name="virtual_joint">
-            <command_interface name="position"/>
-            <state_interface name="position"/>
-            <state_interface name="velocity"/>
-            <state_interface name="effort"/>
-        </joint>
+        <!-- <joint name="virtual_joint"> -->
+            <!-- <command_interface name="position"/> -->
+            <!-- <state_interface name="position"/> -->
+            <!-- <state_interface name="velocity"/> -->
+            <!-- <state_interface name="effort"/> -->
+        <!-- </joint> -->
     </ros2_control>
     <!-- <gazebo> -->
@@ -361,5 +361,5 @@
     <gazebo reference="gps_link">
         <sensor name="gps" type="gps">
-        <update_rate>5</update_rate>
+        <update_rate>10</update_rate>
         <always_on>true</always_on>
         <visualize>false</visualize>
@@ -411,5 +411,5 @@
           <topic>/gps</topic>
           <linkName>gps_link</linkName>
-          <update_rate>5</update_rate>
+          <update_rate>10</update_rate>
           <always_on>true</always_on>
           <gpsNoise>true</gpsNoise>

Commit message: Added a simulated downward camera

File: urdf/custom_iris.xacro (robot description, xacro)
@@ -153,4 +153,10 @@
       <child link="camera_link" />
     </joint>
+    <link name="downward_camera_link"/>
+    <joint name="downward_camera_joint" type="fixed">
+      <origin xyz="0.15 0 -0.01" rpy="0 1.57079632679 0" />
+      <parent link="base_link"/>
+      <child link="downward_camera_link" />
+    </joint>
     <link name="camera_optical_link"/>
     <joint name="camera_optical_joint" type="fixed">
@@ -158,4 +164,10 @@
       <parent link="camera_link"/>
       <child link="camera_optical_link" />
+    </joint>
+    <link name="downward_camera_optical_link"/>
+    <joint name="downward_camera_optical_joint" type="fixed">
+      <origin xyz="0 0 0" rpy="-1.57079632679 0 -1.57079632679"/>
+      <parent link="downward_camera_link"/>
+      <child link="downward_camera_optical_link" />
     </joint>
     <link name="imu_link">
@@ -279,4 +291,37 @@
         <camera_name>camera</camera_name>
         <frame_name>camera_optical_link</frame_name>
+        <hack_baseline>0.07</hack_baseline>
+        <min_depth>0.001</min_depth>
+      </plugin>
+    </sensor>
+    </gazebo>
+    <gazebo reference="downward_camera_link">
+    <sensor type="depth" name="downward_camera">
+        <always_on>true</always_on>
+        <update_rate>10</update_rate>
+        <camera name="downward_camera">
+        <horizontal_fov>1.2</horizontal_fov>
+        <image>
+          <width>640</width>
+          <height>480</height>
+          <format>R8G8B8</format>
+        </image>
+        <depth_camera>
+        </depth_camera>
+        <clip>
+          <near>0.02</near>
+          <far>12</far>
+        </clip>
+        <distortion>
+          <k1>0.0</k1>
+          <k2>0.0</k2>
+          <k3>0.0</k3>
+          <p1>0.0</p1>
+          <p2>0.0</p2>
+        </distortion>
+      </camera>
+      <plugin name="simulated_downward_camera" filename="libgazebo_ros_camera.so">
+        <camera_name>downward_camera</camera_name>
+        <frame_name>downward_camera_optical_link</frame_name>
         <hack_baseline>0.07</hack_baseline>
         <min_depth>0.001</min_depth>
